Commit message: drone description frameworked

File: src/drone_description/urdf/drone_description.urdf (robot description, URDF)
Before this commit: robot None, 0 links, 0 joints
Links:
- added link arm_1; visual box size=0.6 0.2 0.2
- added link arm_2; visual box size=0.6 0.2 0.3
- added link arm_3; visual box size=0.6 0.2 0.4
- added link arm_4; visual box size=0.6 0.2 0.5
- added link base_link; visual box size=0.4 0.1 0.1
- added link prop_1
- added link prop_2
- added link prop_3
- added link prop_4
Joints:
- added joint b_arm_1: type fixed, parent base_link, child arm_1
- added joint b_arm_2: type fixed, parent base_link, child arm_2
- added joint b_arm_3: type fixed, parent base_link, child arm_3
- added joint b_arm_4: type fixed, parent base_link, child arm_4
- added joint m_1: type continuous, parent arm_1, child prop_1
- added joint m_2: type continuous, parent arm_2, child prop_2
- added joint m_3: type continuous, parent arm_3, child prop_3
- added joint m_4: type continuous, parent arm_4, child prop_4
